File: aesir_scale/_autosave-aesir_scale.kicad_sch (KiCad schematic)
At the start: 52 parts, among them J1 jst xh 4, J2 jst gh, J3 jst xh 4, J5 jst gh, J8 USB_C_Receptacle_USB2.0, J9 jst_sh 6, U1 STM32U575CGTx, U2 NAU7802SGI, U3 AZ1117CH2-3.3TRG1, U4 TJA1051T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

Commit message: updated
Parts:
- H1, H2, H3, H4: footprint MountingHole:MountingHole_3.2mm_M3_ISO7380 -> MountingHole:MountingHole_3.2mm_M3_ISO7380_Pad
Changed lines of the file:
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@@
       (effects (font (size 1.27 1.27)) (justify left) hide)
     )
-    (property "Footprint" "MountingHole:MountingHole_3.2mm_M3_ISO7380" (at 127 170.18 0)
+    (property "Footprint" "MountingHole:MountingHole_3.2mm_M3_ISO7380_Pad" (at 127 170.18 0)
       (effects (font (size 1.27 1.27)) hide)
     )
@@
       (effects (font (size 1.27 1.27)) (justify left) hide)
     )
-    (property "Footprint" "MountingHole:MountingHole_3.2mm_M3_ISO7380" (at 135.89 170.18 0)
+    (property "Footprint" "MountingHole:MountingHole_3.2mm_M3_ISO7380_Pad" (at 135.89 170.18 0)
       (effects (font (size 1.27 1.27)) hide)
     )
@@
       (effects (font (size 1.27 1.27)) (justify left) hide)
     )
-    (property "Footprint" "MountingHole:MountingHole_3.2mm_M3_ISO7380" (at 107.95 170.18 0)
+    (property "Footprint" "MountingHole:MountingHole_3.2mm_M3_ISO7380_Pad" (at 107.95 170.18 0)
       (effects (font (size 1.27 1.27)) hide)
     )
@@
       (effects (font (size 1.27 1.27)) (justify left) hide)
     )
-    (property "Footprint" "MountingHole:MountingHole_3.2mm_M3_ISO7380" (at 116.84 170.18 0)
-      (effects (font (size 1.27 1.27)) hide)
-    )
+    (property "Footprint" "MountingHole:MountingHole_3.2mm_M3_ISO7380_Pad" (at 116.84 170.18 0)
+      (effects (font (size 1.27 1.27)) hide)
+    )
